File: PCB/RP0-HandHeld.kicad_sch (KiCad schematic)
At the start: 0 parts

Commit message: Created PCB schematic
Parts:
- added C1, C2: 0.01 uf, symbol Device:C
- added C3, C4: 10 uf, symbol Device:C_Polarized
- added J1: AudioJack2, symbol Connector_Audio:AudioJack2
- added R1, R2: 150 Ohm, symbol Device:R
- added R3, R4: 270 Ohm, symbol Device:R
- added SW1, SW10, SW2, SW3, SW4, SW5, SW6, SW7, SW8, SW9: SW_Push, symbol Switch:SW_Push
- added U1: RASPBERRY_PI_ZERO_2_W, RASPBERRY_PI_ZERO_2_W:MODULE_RASPBERRY_PI_ZERO_2_W, symbol RASPBERRY_PI_ZERO_2_W:RASPBERRY_PI_ZERO_2_W
Connections:
- new net: C1.1, C2.1, R1.1, R2.1, U1.9 (GND_9)
- new net: C2.2, C4.2, R2.2, R4.1
- new net: R4.2, U1.33 (GPIO13)
- new net: SW10.2, U1.5 (GPIO3/SCL)
- new net: SW7.1, U1.40 (GPIO21)
- new net: R3.2, U1.12 (GPIO18/GPIO_GEN1)
- new net: SW8.1, U1.15 (GPIO22/GPIO_GEN3)
- new net: SW4.2, U1.26 (GPIO7/SPI_~{CE1})
- new net: SW2.2, U1.29 (GPIO5)
- new net: SW9.2, U1.3 (GPIO2/SDA1)
- new net: SW3.2, U1.31 (GPIO6)
- new net: SW5.1, U1.35 (GPIO19)
- new net: SW6.1, U1.38 (GPIO20)
- new net: SW1.2, U1.7 (GPIO4/GPIO_GCLK)
- new net: C1.2, C3.2, R1.2, R3.1
- new net: C3.1, J1.T
- new net: C4.1, J1.S
- new net +5V: U1.2 (5V_2)
- new net GND: SW1.1, SW10.1, SW2.1, SW3.1, SW4.1, SW5.2, SW6.2, SW7.2, SW8.2, SW9.1, U1.6 (GND_6)

Commit message: Started working on the pcb
Parts:
- removed J1: AudioJack2, symbol Connector_Audio:AudioJack2
- removed SW1, SW10, SW2, SW3, SW4, SW5, SW6, SW7, SW8, SW9: SW_Push, symbol Switch:SW_Push
- added J1, J10, J11, J12, J13, J2, J3, J4, J5, J6, J7, J8, J9: Conn_01x01_Pin, Connector_Wire:SolderWire-0.5sqmm_1x01_D0.9mm_OD2.3mm, symbol Connector:Conn_01x01_Pin
- C1, C2: footprint (none) -> Capacitor_THT:C_Disc_D5.0mm_W2.5mm_P5.00mm
- C3, C4: footprint (none) -> Capacitor_THT:CP_Radial_D4.0mm_P2.00mm
- R1, R2, R3, R4: footprint (none) -> Resistor_THT:R_Axial_DIN0414_L11.9mm_D4.5mm_P15.24mm_Horizontal
Connections:
- net GND: now also J13.1 (Pin_1)
- net at U1.5 (GPIO3/SCL): now also J11.1 (Pin_1)
- net at U1.40 (GPIO21): now also J5.1 (Pin_1)
- net at U1.15 (GPIO22/GPIO_GEN3): now also J6.1 (Pin_1)
- net at U1.26 (GPIO7/SPI_~{CE1}): now also J7.1 (Pin_1)
- net at U1.29 (GPIO5): now also J9.1 (Pin_1)
- net at U1.3 (GPIO2/SDA1): now also J12.1 (Pin_1)
- net at U1.31 (GPIO6): now also J8.1 (Pin_1)
- net at U1.35 (GPIO19): now also J3.1 (Pin_1)
- net at U1.38 (GPIO20): now also J4.1 (Pin_1)
- net at U1.7 (GPIO4/GPIO_GCLK): now also J10.1 (Pin_1)
- net at C3.1: now also J1.1 (Pin_1)
- net at C4.1: now also J2.1 (Pin_1)
