File: PCB/RP0-HandHeld.kicad_pcb (KiCad board)
At the start: 2 copper layers, 22 parts, among them J1 Conn_01x01_Pin, J10 Conn_01x01_Pin, J11 Conn_01x01_Pin, J12 Conn_01x01_Pin, J13 Conn_01x01_Pin, J2 Conn_01x01_Pin, J3 Conn_01x01_Pin, J4 Conn_01x01_Pin, J5 Conn_01x01_Pin, J6 Conn_01x01_Pin, J7 Conn_01x01_Pin, J8 Conn_01x01_Pin, J9 Conn_01x01_Pin, U1 RASPBERRY_PI_ZERO_2_W

Commit message: Finished PCB
Parts:
- moved J2 144.5 mm to (201.0, 120.0)
- moved J1 143.6 mm to (201.0, 109.0)
- moved R4 125.0 mm to (163.4, 120.0)
- moved R3 124.4 mm to (163.0, 109.0)
- moved C4 123.5 mm to (194.0, 120.0), turned to 180 degrees
- moved C3 122.8 mm to (194.0, 109.0), turned to 180 degrees
- moved J13 101.0 mm to (164.0, 133.0)
- moved J10 99.5 mm to (160.0, 133.0)
- moved J11 96.7 mm to (156.0, 133.0)
- moved J7 92.0 mm to (148.0, 133.0)
- moved J12 91.2 mm to (152.0, 133.0)
- moved J4 89.8 mm to (144.0, 133.0)
- moved J5 84.8 mm to (140.0, 133.0)
- moved J3 83.8 mm to (136.0, 133.0)
- moved J8 75.6 mm to (132.0, 133.0)
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Routing:
- net Net-(J10-Pin_1): track 0.00 -> 175.7 mm
- net Net-(J11-Pin_1): track 0.00 -> 167.9 mm
- net Net-(J12-Pin_1): track 0.00 -> 160.4 mm
- net Net-(J6-Pin_1): track 0.00 -> 118.7 mm
- net Net-(U1-GPIO13): track 0.00 -> 110.9 mm, vias 0 -> 2
- net Net-(J9-Pin_1): track 0.00 -> 98.7 mm
- net Net-(J8-Pin_1): track 0.00 -> 94.4 mm
- net GND: track 0.00 -> 92.9 mm, vias 0 -> 2
- net Net-(J3-Pin_1): track 0.00 -> 86.3 mm
- net Net-(J7-Pin_1): track 0.00 -> 82.8 mm
- net Net-(J4-Pin_1): track 0.00 -> 75.6 mm
- net Net-(J5-Pin_1): track 0.00 -> 74.6 mm
- net Net-(U1-GPIO18/GPIO_GEN1): track 0.00 -> 60.1 mm, vias 0 -> 2
- net Net-(C2-Pad2): track 31.9 -> 91.7 mm
- net Net-(C1-Pad2): track 33.3 -> 71.9 mm
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Other:
- board outline added: 88 x 97 mm

Commit message: Redesigned the PCB
Parts:
- moved C4 59.7 mm to (139.5, 95.5), turned to 0 degrees
- moved C3 58.4 mm to (139.5, 88.0), turned to 0 degrees
- moved J2 38.3 mm to (181.5, 87.0)
- moved J1 36.2 mm to (181.5, 78.5)
- moved R4 31.5 mm to (164.6, 88.5), turned to 180 degrees
- moved J10 28.5 mm to (160.0, 104.5)
- moved J11 28.5 mm to (156.0, 104.5)
- moved J12 28.5 mm to (152.0, 104.5)
- moved J13 28.5 mm to (164.0, 104.5)
- moved J3 28.5 mm to (136.0, 104.5)
- moved J4 28.5 mm to (144.0, 104.5)
- moved J5 28.5 mm to (140.0, 104.5)
- moved J6 28.5 mm to (124.0, 104.5)
- moved J7 28.5 mm to (148.0, 104.5)
- moved J8 28.5 mm to (132.0, 104.5)
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Routing:
- net Net-(J1-Pin_1): track 7.00 -> 62.2 mm
- net GND: track 92.9 -> 39.5 mm, vias 2 -> 1
- net Net-(U1-GPIO13): track 110.9 -> 64.4 mm
- net Net-(U1-GND_9): track 149.7 -> 104.0 mm
- net Net-(J10-Pin_1): track 175.7 -> 132.9 mm
- net Net-(J2-Pin_1): track 7.00 -> 48.3 mm
- net Net-(J12-Pin_1): track 160.4 -> 121.3 mm
- net Net-(J11-Pin_1): track 167.9 -> 129.2 mm
- net Net-(J9-Pin_1): track 98.7 -> 68.2 mm
- net Net-(J6-Pin_1): track 118.7 -> 88.3 mm
- net Net-(J8-Pin_1): track 94.4 -> 64.9 mm
- net Net-(J4-Pin_1): track 75.6 -> 46.7 mm
- net Net-(J3-Pin_1): track 86.3 -> 57.7 mm
- net Net-(J5-Pin_1): track 74.6 -> 46.1 mm
- net Net-(J7-Pin_1): track 82.8 -> 54.3 mm
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Other:
- board size 88 x 97 mm -> 69.5 x 68.5 mm

Commit message: Edited silkscreen PCB
Other:
- board text added: "150 Ohm"
- board text added: "270 Ohm"
- board text added: ":D"
- board text added: "GameBoy Pro Max"
- board text added: "Ondkos"
- board text added: "RP0-HandHeld"
- board text added: "https://github.com/OndrejVacekSPSCL/RP0-HandHeld"
Changed lines of the file:
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@@
 		(tags "connector wire 0.5sqmm")
 		(property "Reference" "J8"
-			(at 0 -2.35 0)
+			(at -1 -2.35 0)
 			(layer "F.SilkS")
+			(hide yes)
 			(effects
 				(font
@@
 		(tags "C Disc series Radial pin pitch 5.00mm diameter 5mm width 2.5mm Capacitor")
 		(property "Reference" "C2"
-			(at 2.5 -2.5 90)
+			(at 2.5 0 90)
 			(layer "F.SilkS")
 			(effects
@@
 		(tags "connector wire 0.5sqmm")
 		(property "Reference" "J6"
-			(at 0 -2.35 0)
+			(at -1 -2.35 0)
 			(layer "F.SilkS")
+			(hide yes)
 			(effects
 				(font
@@
 		(tags "connector wire 0.5sqmm")
 		(property "Reference" "J13"
-			(at 0 -2.35 0)
+			(at -1.5 -2.35 0)
 			(layer "F.SilkS")
+			(hide yes)
 			(effects
 				(font
@@
 		(tags "connector wire 0.5sqmm")
 		(property "Reference" "J3"
-			(at 0 -2.35 0)
+			(at -1 -2.35 0)
 			(layer "F.SilkS")
+			(hide yes)
 			(effects
 				(font
@@
 		(tags "connector wire 0.5sqmm")
 		(property "Reference" "J11"
-			(at 0 -2.35 0)
+			(at -1.5 -2.35 0)
 			(layer "F.SilkS")
+			(hide yes)
 			(effects
 				(font
@@
 			(at 0 -2.35 0)
 			(layer "F.SilkS")
+			(hide yes)
 			(effects
 				(font
@@
 		(tags "Resistor Axial_DIN0414 series Axial Horizontal pin pitch 15.24mm 2W length 11.9mm diameter 4.5mm")
 		(property "Reference" "R4"
-			(at 7.62 -3.37 0)
+			(at 12.62 1.5 0)
 			(layer "F.SilkS")
 			(effects
@@
 		(tags "connector wire 0.5sqmm")
 		(property "Reference" "J9"
-			(at 0 -2.35 0)
+			(at -1 -2.35 0)
 			(layer "F.SilkS")
+			(hide yes)
 			(effects
 				(font
@@
 		(tags "connector wire 0.5sqmm")
 		(property "Reference" "J5"
-			(at 0 -2.35 0)
+			(at -1 -2.35 0)
 			(layer "F.SilkS")
+			(hide yes)
 			(effects
 				(font
@@
 		(tags "Resistor Axial_DIN0414 series Axial Horizontal pin pitch 15.24mm 2W length 11.9mm diameter 4.5mm")
 		(property "Reference" "R1"
-			(at 7.62 -3.37 0)
+			(at 2.62 -1.5 0)
 			(layer "F.SilkS")
 			(effects
@@
 			(at 0 -2.35 0)
 			(layer "F.SilkS")
+			(hide yes)
 			(effects
 				(font
@@
 			(at 0 -2.35 0)
 			(layer "F.SilkS")
+			(hide yes)
 			(effects
 				(font
@@
 			(at 0 -2.35 0)
 			(layer "F.SilkS")
+			(hide yes)
 			(effects
 				(font
@@
 		(tags "C Disc series Radial pin pitch 5.00mm diameter 5mm width 2.5mm Capacitor")
 		(property "Reference" "C1"
-			(at 2.5 -2.5 90)
+			(at 3 0.5 90)
 			(layer "F.SilkS")
 			(effects
@@
 		(tags "connector wire 0.5sqmm")
 		(property "Reference" "J4"
-			(at 0 -2.35 0)
+			(at -2 -2 0)
 			(layer "F.SilkS")
+			(hide yes)
 			(effects
 				(font
@@
 			(at 0 -2.35 0)
 			(layer "F.SilkS")
+			(hide yes)
 			(effects
 				(font
@@
 		(tags "Resistor Axial_DIN0414 series Axial Horizontal pin pitch 15.24mm 2W length 11.9mm diameter 4.5mm")
 		(property "Reference" "R3"
-			(at 7.62 -3.37 0)
+			(at 12.62 1.5 0)
 			(layer "F.SilkS")
 			(effects
@@
 		(at 148 53.5 180)
 		(property "Reference" "U1"
-			(at -29.569 -17.0132 0)
+			(at -12 -6 0)
 			(layer "F.SilkS")
+			(hide yes)
 			(effects
 				(font
@@
 		(tags "CP Radial series Radial pin pitch 2.00mm diameter 4mm height 7mm Electrolytic Capacitor")
 		(property "Reference" "C4"
-			(at 1 -3.25 0)
+			(at -0.527401 -3 0)
 			(layer "F.SilkS")
 			(effects
@@
 		(tags "Resistor Axial_DIN0414 series Axial Horizontal pin pitch 15.24mm 2W length 11.9mm diameter 4.5mm")
 		(property "Reference" "R2"
-			(at 7.62 -3.37 0)
+			(at 2.62 -1.5 0)
 			(layer "F.SilkS")
 			(effects
@@
 		(layer "Edge.Cuts")
 	)
+	(gr_text "GameBoy Pro Max"
+		(at 119 90.5 90)
+		(layer "F.SilkS")
+		(effects
+			(font
+				(size 1 1)
+				(thickness 0.15)
+			)
+			(justify left bottom)
+		)
+	)
+	(gr_text ":D\n"
+		(at 181.5 70.5 0)
+		(layer "F.SilkS")
+		(effects
+			(font
+				(size 1 1)
+				(thickness 0.1)
+			)
+			(justify left bottom)
+		)
+	)
+	(gr_text "Ondkos"
+		(at 177.5 105.5 0)
+		(layer "F.SilkS")
+		(effects
+			(font
+				(size 1 1)
+				(thickness 0.1)
+			)
+			(justify left bottom)
+		)
+	)
+	(gr_text "150 Ohm"
+		(at 154 82.5 0)
+		(layer "F.SilkS")
+		(effects
+			(font
+				(size 1 1)
+				(thickness 0.1)
+			)
+			(justify left bottom)
+		)
+	)
+	(gr_text "150 Ohm\n"
+		(at 153.5 76 0)
+		(layer "F.SilkS")
+		(effects
+			(font
+				(size 1 1)
+				(thickness 0.1)
+			)
+			(justify left bottom)
+		)
+	)
+	(gr_text "270 Ohm"
+		(at 154.5 95.5 0)
+		(layer "F.SilkS")
+		(effects
+			(font
+				(size 1 1)
+				(thickness 0.1)
+			)
+			(justify left bottom)
+		)
+	)
+	(gr_text "https://github.com/OndrejVacekSPSCL/RP0-HandHeld"
+		(at 157.5 68 0)
+		(layer "F.SilkS")
+		(effects
+			(font
+				(size 0.5 0.5)
+				(thickness 0.05)
+			)
+			(justify left bottom)
+		)
+	)
+	(gr_text "RP0-HandHeld\n"
+		(at 124.5 43 0)
+		(layer "F.SilkS")
+		(effects
+			(font
+				(size 1 1)
+				(thickness 0.1)
+			)
+			(justify left bottom)
+		)
+	)
+	(gr_text "270 Ohm"
+		(at 154 89 0)
+		(layer "F.SilkS")
+		(effects
+			(font
+				(size 1 1)
+				(thickness 0.1)
+			)
+			(justify left bottom)
+		)
+	)
 	(segment
